File: ModuleV490-AllInOne/Module_16S.kicad_sch (KiCad schematic)
At the start: 59 parts, among them J14 BALANCE BOARD, J15 BALANCE BOARD, J6 CELL CONNECTOR PLUG, J7 CELL CONNECTOR, U1 MAX14921ECS+T, U2 MCP1501-40xSN, U3 MCP33151-05-E/MS, U6 MCP1502T-45E/CHY

Commit message: Swap V reference chip to Texas Instruments REF5045AIDR (fixed 4.5V)
Parts:
- removed C24: 100pF, Capacitor_SMD:C_0603_1608Metric, symbol Device:C
- removed R52: 100R, Resistor_SMD:R_0603_1608Metric, symbol Device:R
- removed U2: MCP1501-40xSN, Package_SO:SOIC-8_3.9x4.9mm_P1.27mm, symbol Reference_Voltage:MCP1501-40xSN
- removed U6: MCP1502T-45E/CHY, Package_TO_SOT_SMD:SOT-23-6, symbol mcp1502t-45e:MCP1502T-45E
- added C26: 1uF, Capacitor_SMD:C_0805_2012Metric, symbol Device:C
- added U7: REF5045AIDR, Package_SO:SOIC-8_3.9x4.9mm_P1.27mm, symbol Reference_Voltage:REF5045AD
- TP4: value TEST_4096 -> TEST_VREF
Connections:
- net +5V: now also C26.2, U7.2 (Vin); no longer C27.2
- net GND: now also C26.1, U7.4 (GND)
- net VREF4096 renamed VREF
- net VREF: now also C27.2, U7.6 (Vout)
- no-connect marks 20 -> 22
Other:
- moved on the sheet: C27, TP4
